File: first_punch.kicad_sch (KiCad schematic)
At the start: 67 parts, among them J1 AudioJack3, J2 Barrel_Jack_Switch, Q1 2N3904, SW1 SMTS-102, SW2 SMTS-102, SW3 SMTS-102, U1 40106, U3 LM358

Commit message: Finish circuit and pcb
Parts:
- removed J1: AudioJack3, Import:PJ302M, symbol Connector_Audio:AudioJack3
- added D9: LED, LED_THT:LED_D5.0mm, symbol Device:LED
- added J3: ~, Import:PJ302M, symbol import:AudioJackMono
- added R27: 10k, Resistor_THT:R_Axial_DIN0207_L6.3mm_D2.5mm_P10.16mm_Horizontal, symbol Device:R
- SW1, SW2, SW3: footprint V:SIP3 -> Import:SMTS-102
Connections:
- net +12V: now also D9.2 (A)
- net GND: now also RV4.1, J3.1, R27.2; no longer RV4.3
- net at D6.2 (A), RV1.2, SW2.2 (B)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: now also RV1.1; no longer RV1.3
- net at C14.1: now also J3.3
- net at R7.2: now also RV5.3; no longer RV5.1
- net at D7.2 (A), RV6.2, SW1.2 (B)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: now also RV6.1; no longer RV6.3
- net at R13.1, RV2.2, RV7.3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: now also RV2.1; no longer RV2.3
- net at Q1.3 (C), R11.2, RV5.2: now also RV5.1; no longer RV5.3
- net at SW1.3 (C): now also RV4.3; no longer RV4.1
- net at RV3.1: now also D8.2 (A), RV3.2, SW3.2 (B), U1.6; no longer R3.2
- net at R1.2: now also RV1.3; no longer RV1.1
- net at R2.2: now also RV6.3; no longer RV6.1
- net at R8.2: now also RV2.3; no longer RV2.1
- new net: D9.1 (K), R27.1
- new net: R3.2, RV3.3
Other:
- note added: "CW to 3 CCW to 1"
- note added: "For cd40106 Vo=13.5 Vdd=15 min Io=3.4 typ Io=6.8"
- moved on the sheet: RV1, RV2, RV3, RV5, RV6

Commit message: change AudioJack to PJ-316 Separate leds into green and red
Parts:
- D6, D7, D8: value LED -> LED green
- D9: value LED -> LED red
- J3: footprint Import:PJ302M -> Import:PJ-316
Changed lines of the file:
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@@
       (effects (font (size 1.27 1.27)))
     )
-    (property "Value" "LED" (at 60.0075 24.765 0)
+    (property "Value" "LED green" (at 60.0075 24.765 0)
       (effects (font (size 1.27 1.27)))
     )
@@
       (effects (font (size 1.27 1.27)))
     )
-    (property "Value" "LED" (at 60.0075 64.135 0)
+    (property "Value" "LED green" (at 60.0075 64.135 0)
       (effects (font (size 1.27 1.27)))
     )
@@
       (effects (font (size 1.27 1.27)))
     )
-    (property "Footprint" "Import:PJ302M" (at 255.27 91.44 0)
+    (property "Footprint" "Import:PJ-316" (at 255.27 91.44 0)
       (effects (font (size 1.27 1.27)) hide)
     )
@@
       (effects (font (size 1.27 1.27)))
     )
-    (property "Value" "LED" (at 61.2775 117.475 0)
+    (property "Value" "LED green" (at 61.2775 117.475 0)
       (effects (font (size 1.27 1.27)))
     )
@@
       (effects (font (size 1.27 1.27)) (justify right))
     )
-    (property "Value" "LED" (at 71.755 173.0375 90)
+    (property "Value" "LED red" (at 71.755 173.0375 90)
       (effects (font (size 1.27 1.27)) (justify right))
     )
