File: first_ufo_v1/first_punch.kicad_sch (KiCad schematic)
At the start: 69 parts, among them J2 Barrel_Jack_Switch, Q1 2N3904, SW1 SMTS-102, SW2 SMTS-102, SW3 SMTS-102, U1 40106, U3 LM358

Commit message: move to directory
Other:
- note added: "RV12 = 0 Hi freq RV12 = 1Meg low freq"
- moved on the sheet: R21, RV11
Changed lines of the file:
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@@
 (kicad_sch (version 20230121) (generator eeschema)
   (paper "A4")
+  (junction (at 248.92 31.75) (diameter 0) (color 0 0 0 0)
+  )
   (junction (at 55.88 120.65) (diameter 0) (color 0 0 0 0)
   )
   (junction (at 115.57 185.42) (diameter 0) (color 0 0 0 0)
   )
+  (junction (at 256.54 31.75) (diameter 0) (color 0 0 0 0)
+  )
   (junction (at 54.61 41.91) (diameter 0) (color 0 0 0 0)
   )
@@
   (junction (at 21.59 81.28) (diameter 0) (color 0 0 0 0)
   )
-  (junction (at 248.92 29.21) (diameter 0) (color 0 0 0 0)
-  )
   (junction (at 55.88 134.62) (diameter 0) (color 0 0 0 0)
   )
@@
   (junction (at 170.18 58.42) (diameter 0) (color 0 0 0 0)
   )
-  (junction (at 256.54 19.05) (diameter 0) (color 0 0 0 0)
-  )
   (junction (at 172.72 52.07) (diameter 0) (color 0 0 0 0)
   )
@@
   (junction (at 118.11 109.22) (diameter 0) (color 0 0 0 0)
   )
-  (junction (at 248.92 19.05) (diameter 0) (color 0 0 0 0)
-  )
   (junction (at 22.86 134.62) (diameter 0) (color 0 0 0 0)
   )
+  (junction (at 248.92 22.86) (diameter 0) (color 0 0 0 0)
+  )
   (junction (at 156.21 175.26) (diameter 0) (color 0 0 0 0)
   )
@@
     (stroke (width 0) (type default))
   )
-  (wire (pts (xy 259.08 19.05) (xy 256.54 19.05))
+  (wire (pts (xy 259.08 31.75) (xy 256.54 31.75))
+    (stroke (width 0) (type default))
+  )
+  (wire (pts (xy 248.92 22.86) (xy 248.92 19.05))
     (stroke (width 0) (type default))
   )
@@
     (stroke (width 0) (type default))
   )
-  (wire (pts (xy 246.38 31.75) (xy 246.38 29.21))
-    (stroke (width 0) (type default))
-  )
   (wire (pts (xy 172.72 52.07) (xy 181.61 52.07))
     (stroke (width 0) (type default))
@@
     (stroke (width 0) (type default))
   )
-  (wire (pts (xy 246.38 29.21) (xy 248.92 29.21))
+  (wire (pts (xy 246.38 31.75) (xy 248.92 31.75))
     (stroke (width 0) (type default))
   )
@@
     (stroke (width 0) (type default))
   )
-  (wire (pts (xy 248.92 15.24) (xy 252.73 15.24))
+  (wire (pts (xy 248.92 19.05) (xy 252.73 19.05))
     (stroke (width 0) (type default))
   )
@@
     (stroke (width 0) (type default))
   )
+  (wire (pts (xy 248.92 22.86) (xy 248.92 31.75))
+    (stroke (width 0) (type default))
+  )
   (wire (pts (xy 152.4 182.88) (xy 152.4 187.96))
     (stroke (width 0) (type default))
@@
     (stroke (width 0) (type default))
   )
-  (wire (pts (xy 248.92 19.05) (xy 248.92 29.21))
-    (stroke (width 0) (type default))
-  )
   (wire (pts (xy 58.42 181.61) (xy 54.61 181.61))
     (stroke (width 0) (type default))
@@
     (stroke (width 0) (type default))
   )
-  (wire (pts (xy 256.54 29.21) (xy 256.54 19.05))
+  (wire (pts (xy 256.54 31.75) (xy 256.54 22.86))
     (stroke (width 0) (type default))
   )
@@
     (stroke (width 0) (type default))
   )
-  (wire (pts (xy 248.92 19.05) (xy 248.92 15.24))
-    (stroke (width 0) (type default))
-  )
   (wire (pts (xy 101.6 134.62) (xy 100.33 134.62))
     (stroke (width 0) (type default))
@@
     (stroke (width 0) (type default))
   )
-  (wire (pts (xy 259.08 31.75) (xy 259.08 19.05))
-    (stroke (width 0) (type default))
-  )
   (wire (pts (xy 33.02 81.28) (xy 21.59 81.28))
     (stroke (width 0) (type default))
@@
   (wire (pts (xy 123.19 27.94) (xy 123.19 24.13))
     (stroke (width 0) (type default))
+  )
+  (text "RV12 = 0 Hi freq\nRV12 = 1Meg low freq" (at 215.9 25.4 0)
+    (effects (font (size 1.27 1.27)) (justify left bottom))
   )
   (text "CW to 3\nCCW to 1\n" (at 40.64 20.32 0)
     (effects (font (size 1.27 1.27)) (justify left bottom))
   )
-  (text "CW to 3\nCCW to 1\n" (at 226.06 26.67 0)
+  (text "CW to 3\nCCW to 1\n" (at 222.25 19.05 0)
     (effects (font (size 1.27 1.27)) (justify left bottom))
   )
@@
     )
   )
-  (symbol (lib_id "Device:R") (at 252.73 29.21 270) (unit 1)
+  (symbol (lib_id "Device:R") (at 252.73 31.75 270) (unit 1)
     (in_bom yes) (on_board yes) (dnp no) (fields_autoplaced)
-    (property "Reference" "R21" (at 252.73 24.13 90)
-      (effects (font (size 1.27 1.27)))
-    )
-    (property "Value" "470k" (at 252.73 26.67 90)
-      (effects (font (size 1.27 1.27)))
-    )
-    (property "Footprint" "Resistor_THT:R_Axial_DIN0207_L6.3mm_D2.5mm_P10.16mm_Horizontal" (at 252.73 27.432 90)
-      (effects (font (size 1.27 1.27)) hide)
-    )
-    (property "Datasheet" "~" (at 252.73 29.21 0)
+    (property "Reference" "R21" (at 252.73 26.67 90)
+      (effects (font (size 1.27 1.27)))
+    )
+    (property "Value" "470k" (at 252.73 29.21 90)
+      (effects (font (size 1.27 1.27)))
+    )
+    (property "Footprint" "Resistor_THT:R_Axial_DIN0207_L6.3mm_D2.5mm_P10.16mm_Horizontal" (at 252.73 29.972 90)
+      (effects (font (size 1.27 1.27)) hide)
+    )
+    (property "Datasheet" "~" (at 252.73 31.75 0)
       (effects (font (size 1.27 1.27)) hide)
     )
@@
     )
   )
-  (symbol (lib_id "Device:R_Potentiometer") (at 252.73 19.05 90) (unit 1)
+  (symbol (lib_id "Device:R_Potentiometer") (at 252.73 22.86 90) (unit 1)
     (in_bom yes) (on_board yes) (dnp no)
-    (property "Reference" "RV11" (at 246.38 21.59 90)
-      (effects (font (size 1.27 1.27)))
-    )
-    (property "Value" "500k" (at 257.81 21.59 90)
-      (effects (font (size 1.27 1.27)))
-    )
-    (property "Footprint" "Potentiometer_THT:Potentiometer_Bourns_PTV09A-1_Single_Vertical" (at 252.73 19.05 0)
-      (effects (font (size 1.27 1.27)) hide)
-    )
-    (property "Datasheet" "~" (at 252.73 19.05 0)
-      (effects (font (size 1.27 1.27)) hide)
-    )
+    (property "Reference" "RV11" (at 246.38 25.4 90)
+      (effects (font (size 1.27 1.27)))
+    )
+    (property "Value" "500k" (at 257.81 25.4 90)
+      (effects (font (size 1.27 1.27)))
+    )
+    (property "Footprint" "Potentiometer_THT:Potentiometer_Bourns_PTV09A-1_Single_Vertical" (at 252.73 22.86 0)
+      (effects (font (size 1.27 1.27)) hide)
+    )
+    (property "Datasheet" "~" (at 252.73 22.86 0)
+      (effects (font (size 1.27 1.27)) hide)
+    )
