File: first_ufo_v1_1/first_ufo_v1_1.kicad_pcb (KiCad board)
At the start: 2 copper layers, 141 x 99.1 mm, 74 parts, among them J2 Barrel_Jack_Switch, Q1 2N3904, SW1 SMTS-102, SW2 SMTS-102, SW3 SMTS-102, U1 40106, U3 LM358

Commit message: no message
Parts:
- removed R12, R13, R14: 100k, Resistor_THT:R_Axial_DIN0207_L6.3mm_D2.5mm_P10.16mm_Horizontal
- removed R21: 470k, Resistor_THT:R_Axial_DIN0207_L6.3mm_D2.5mm_P10.16mm_Horizontal
- removed REF** (x4): MountingHole_3.2mm_M3, MountingHole:MountingHole_3.2mm_M3
- removed REF**: Polarity_Center_Positive_6mm_SilkScreen, Symbol:Polarity_Center_Positive_6mm_SilkScreen
- added H1: MountingHole, MountingHole:MountingHole_3.2mm_M3, F.Cu at (168.9, 40.6)
- added H2: MountingHole, MountingHole:MountingHole_3.2mm_M3, F.Cu at (168.9, 129.5)
- added H3: MountingHole, MountingHole:MountingHole_3.2mm_M3, F.Cu at (38.1, 129.5)
- added H4: MountingHole, MountingHole:MountingHole_3.2mm_M3, F.Cu at (38.1, 40.6)
- added LO1: ~, Import:Polarity_Center_Positive_3mm_SilkScreen, F.Cu at (170.8, 52.1)
- added RV10: 1M, Potentiometer_THT:Potentiometer_Bourns_PTV09A-1_Single_Vertical, F.Cu at (128.9, 79.0)
- C11, C12: value 470p -> 1n
- R1, R15, R16, R17, R2, R3: value 4k7 -> 27k
- R18: value 1k -> 4k7
- R20: value 10M -> 4M7
- R8: value 4k7 -> 10k
- RV11: value 500k -> 100k
- RV12, RV7, RV8, RV9: value 1M -> 100k
- moved SW2 26.1 mm to (59.1, 66.7)
- moved D2 21.5 mm to (38.7, 48.9), turned to -90 degrees
- moved R9 13.6 mm to (99.1, 98.4), turned to 180 degrees
- moved SW3 12.2 mm to (51.4, 98.4)
- moved R15 11.8 mm to (110.5, 76.0)
- moved R5 10.4 mm to (130.2, 72.4)
- moved R16 10.2 mm to (110.5, 79.2)
- moved D1 10.2 mm to (99.1, 101.6), turned to 180 degrees
- moved C7 9.44 mm to (121.9, 79.8), turned to 180 degrees
- moved C8 9.19 mm to (79.4, 61.0)
- moved R17 8.82 mm to (110.5, 82.3)
- moved R19 8.71 mm to (130.2, 67.9)
- moved R6 8.64 mm to (130.2, 75.6)
- moved C5 8.17 mm to (40.1, 99.1)
- moved C6 7.25 mm to (121.9, 82.3)
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Connections:
- R22 pad 2: Net-(C13-Pad2) -> Net-(R22-Pad2)
- RV7 pad 1: unconnected-(RV7-Pad1) -> GND
- RV8 pad 1: unconnected-(RV8-Pad1) -> GND
- RV9 pad 1: unconnected-(RV9-Pad1) -> GND
Routing:
- net GND: track 342.0 -> 151.6 mm, vias 1 -> 0
- net +12V: track 169.3 -> 8.48 mm, vias 1 -> 0
- net Net-(R10-Pad1): track 122.1 -> 9.46 mm
- net Net-(D7-A): track 117.6 -> 13.3 mm
- net Net-(D1-K): track 98.5 -> 0.00 mm
- net Net-(C4-Pad1): track 98.8 -> 5.61 mm
- net Net-(R16-Pad2): track 88.5 -> 0.00 mm
- net Net-(R11-Pad1): track 80.1 -> 0.00 mm
- net Net-(SW1-C): track 70.6 -> 0.00 mm
- net Net-(D6-A): track 61.8 -> 2.50 mm
- net Net-(RV2-Pad1): track 71.4 -> 12.7 mm
- net Net-(C12-Pad2): track 56.0 -> 0.00 mm
- net Net-(R19-Pad1): track 56.2 -> 2.50 mm
- net Net-(U3A--): track 53.2 -> 0.00 mm
- net Net-(U3B--): track 48.8 -> 0.00 mm
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Other:
- board text added: "DEPTH"
- board text added: "FILTER"
- board text added: "FIRST UFO"
- board text added: "FREQ"
- board text added: "LPF"
- board text added: "RES"
- board text added: "TOUCH!"
- board text added: "VOLUME"
- board text removed: "Amount"
- board text removed: "Cutoff Filter"
- board text removed: "First UFO"
- board text removed: "Freq"
- board text removed: "Res"
- board text removed: "Touch!"
- board text removed: "Ver1"
- board text removed: "Volume"

Commit message: move lines
Parts:
- moved R16 64.4 mm to (169.5, 104.8)
- moved R9 64.2 mm to (163.2, 94.6)
- moved D1 63.8 mm to (161.9, 90.8)
- moved R17 57.5 mm to (53.3, 88.9)
- moved RV6 46.7 mm to (99.8, 88.6)
- moved R18 34.4 mm to (97.2, 48.9)
- moved R20 34.4 mm to (97.2, 52.1)
- moved RV10 32.0 mm to (158.8, 67.6)
- moved C11 31.9 mm to (100.4, 40.0)
- moved C12 31.9 mm to (100.4, 42.5)
- moved C13 31.9 mm to (100.4, 45.1)
- moved R26 28.6 mm to (42.5, 93.3)
- moved R15 24.7 mm to (87.6, 66.7)
- moved SW1 24.7 mm to (102.3, 83.8)
- moved C6 24.4 mm to (100.9, 69.8)
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Routing:
- net GND: track 151.6 -> 61.7 mm
- net Net-(D5-Pad2): track 51.7 -> 0.00 mm
- net Net-(D3-K): track 27.5 -> 0.00 mm
- net Net-(D3-A): track 25.3 -> 0.00 mm
- net Net-(R2-Pad2): track 23.9 -> 0.00 mm
- net Net-(Q1-C): track 21.1 -> 2.50 mm
- net Net-(Q1-B): track 15.5 -> 0.00 mm
- net Net-(D7-A): track 13.3 -> 0.00 mm
- net Net-(R10-Pad1): track 9.46 -> 0.00 mm
- net Net-(R7-Pad2): track 6.13 -> 0.00 mm
- net Net-(D9-K): track 5.61 -> 0.00 mm
- net +12V: track 8.48 -> 4.89 mm
Other:
- board text added: "OUT"
- board text added: "VOL"
- board text removed: "LPF"
- board text removed: "VOLUME"

Commit message: many many changes
Parts:
- D5: footprint Import:tactile pad triangle -> Import:tactile pad triangle_1
- moved D5 8.94 mm to (127.0, 123.4)
- moved C2 7.75 mm to (149.9, 78.2)
- moved D4 6.38 mm to (151.8, 69.8)
- moved C1 5.43 mm to (61.0, 75.6)
- moved U1 5.43 mm to (40.6, 83.2)
- moved C3 2.29 mm to (62.9, 67.3)
- moved R15 1.91 mm to (87.6, 64.8)
- moved R19 1.27 mm to (110.5, 67.9)
- moved R22 1.27 mm to (107.3, 67.9)
- moved R27 1.02 mm to (167.1, 65.0)
- moved C14 0.90 mm to (138.5, 61.0)
- moved C8 0.90 mm to (80.0, 60.3)
Routing:
- net GND: track 61.7 -> 425.9 mm
- net Net-(U3A--): track 0.00 -> 182.4 mm
- net +12V: track 4.89 -> 155.7 mm
- net Net-(D1-K): track 0.00 -> 140.4 mm
- net Net-(R10-Pad1): track 0.00 -> 123.0 mm
- net Net-(D7-A): track 0.00 -> 110.0 mm
- net Net-(C4-Pad1): track 5.61 -> 103.8 mm
- net Net-(SW1-C): track 0.00 -> 77.1 mm
- net Net-(D3-K): track 0.00 -> 72.6 mm
- net Net-(C12-Pad2): track 0.00 -> 71.6 mm
- net Net-(D2-K): track 0.00 -> 70.2 mm
- net Net-(D6-A): track 2.50 -> 71.6 mm
- net Net-(C13-Pad2): track 0.00 -> 67.6 mm
- net Net-(R11-Pad1): track 0.00 -> 63.9 mm
- net Vref: track 0.00 -> 62.9 mm
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Other:
- board text added: "Block diagram"
- board text added: "FIRST"
- board text added: "OSC"
- board text added: "Schmitt Trigger CD40106B"
- board text added: "TOUCH"
- board text added: "UFO"
- board text added: "original circuit on github.com/paltus23/first_punch"
- board text removed: "FIRST UFO"
- board text removed: "original circuit on github.com/paltus23/first_ufo_v1_1"

Commit message: no message
Other:
- board text removed: "Schmitt Trigger CD40106B"
